File: kicad_project/SmartCruiseControl/SmartCruiseControl.kicad_pcb (KiCad board)
At the start: 2 copper layers, 80 x 80 mm, 47 parts, among them J1 USB 5V, J2 CAN bus, J3 Buttons + led, J4 Accelerator pedal, J5 Brake + clutch, K1 HK19F-DC 5V-SHG, Q1 2N3904, Q2 2N3904, Q3 2N3904, Q4 2N3904, Q5 IRLZ44N, U1 SN65HVD230, U2 ESP32DevKitv1

Commit message: Updated board version to v1.1.1
Increased hole size from M2 to M3
Parts:
- H1, H2, H3, H4: footprint MountingHole:MountingHole_2.2mm_M2_Pad_Via -> MountingHole:MountingHole_3.2mm_M3_Pad_Via
- J5: value Brake + clutch -> Brake+clutch
- moved J1 0.80 mm to (113.5, 60.0)
- moved J2 0.60 mm to (127.5, 59.9)
- moved J3 0.60 mm to (144.0, 59.9)
- moved J4 0.60 mm to (158.5, 59.9)
- moved J5 0.40 mm to (168.0, 59.9)
- moved TP4 0.25 mm to (160.5, 65.5)
Other:
- board text added: "SmartCruiseControl v1.1.1"
- board text removed: "SmartCruiseControl v1.1"
