File: kicad_project/SmartCruiseControl/SmartCruiseControl.kicad_sch (KiCad schematic)
At the start: 45 parts, among them J1 Accelerator pedal, J2 CAN bus, J3 Brake + clutch, J4 Buttons + led, J5 USB 5V, K1 HK19F-DC 5V-SHG, Q1 IRLZ44N, Q2 2N3904, Q3 2N3904, Q4 2N3904, Q5 2N3904, U1 SN65HVD230, U2 ESP32DevKitv1

Commit message: Updated board to v1.1
Parts:
- removed TP11: 3.3V, TestPoint:TestPoint_THTPad_D1.5mm_Drill0.7mm, symbol Connector:TestPoint
- removed TP12, TP4: GND, TestPoint:TestPoint_THTPad_2.0x2.0mm_Drill1.0mm, symbol Connector:TestPoint
- added C1: 1uF, Capacitor_THT:CP_Radial_D5.0mm_P2.00mm, symbol Device:C_Polarized
- added C2: 100nF, Capacitor_THT:C_Disc_D5.0mm_W2.5mm_P5.00mm, symbol Device:C
- added TP14: GND, TestPoint:TestPoint_THTPad_2.0x2.0mm_Drill1.0mm, symbol Connector:TestPoint
- added TP3: CAN_L, TestPoint:TestPoint_THTPad_D1.0mm_Drill0.5mm, symbol Connector:TestPoint
- added TP5: CAN_H, TestPoint:TestPoint_THTPad_D1.0mm_Drill0.5mm, symbol Connector:TestPoint
- H1: renamed from H2; KiLib_Generator (none) -> mounting_hardware/mounting_hole
- H2: renamed from H3; KiLib_Generator (none) -> mounting_hardware/mounting_hole
- H3: renamed from H1; KiLib_Generator (none) -> mounting_hardware/mounting_hole
- H4: KiLib_Generator (none) -> mounting_hardware/mounting_hole
- R1: renamed from R11; value 5k -> 5.1k; KiLib_Generator (none) -> resistor/THT
- R10, R6, R9: value 47k -> 100k
- R5: renamed from R7; value 47k -> 100k
- U1: KiLib_Generator (none) -> package/gullwing
- renumbered C1 to C3, C2 to C4, J5 to J1, J4 to J3, J1 to J4, J3 to J5, Q3 to Q1, Q4 to Q2, Q2 to Q3, Q5 to Q4, Q1 to Q5, R8 to R11, R3 to R2, R5 to R3, R1 to R4, R4 to R7, R2 to R8, TP7 to TP10, TP8 to TP11, TP14 to TP12, TP9 to TP2, TP5 to TP4, TP10 to TP6, TP2 to TP7, TP6 to TP8, TP3 to TP9
Connections:
- net +5V: no longer J1.1 (Pin_1), J1.2 (Pin_2), J3.1 (Pin_1), J3.2 (Pin_2)
- net BUTTON_KEY: now also J3.2 (Pin_2), C2.1; no longer J3.4 (Pin_4)
- net CAN_HIGH: now also TP5.1
- net CAN_LOW: now also TP3.1
- net GND: now also C1.2, C2.2, TP14.1
- net 5V_IN: now reaches J3.5 (Pin_5)
- net 5V_IN: now also J1.1 (Pin_1); no longer R3.2
- net RELAY_GND: now reaches D1.2 (A), K1.A2, Q5.2 (D)
- net CAN_TTL_TX: now reaches U1.1 (D), U2.8 (D5)
- net CAN_TTL_RX: now reaches U1.4 (R), U2.5 (D4)
- net PWM_GENERATED_APPS2: now reaches R8.1, U2.10 (D19)
- net RELAY_ENABLE: now reaches R7.1, U2.11 (D21)
- net BRAKE_INPUT: now reaches Q3.3 (C), U2.14 (D22)
- net CLUTCH_INPUT: now reaches Q1.3 (C), U2.15 (D23)
- net EN: now reaches U2.16 (EN)
- net EN: now also C1.1
- net PWM_GENERATED_APPS1: now reaches R4.1, U2.9 (D18)
- new net 5V_OUT: J1.2 (Pin_2), J3.4 (Pin_4)
- new net Net-(J2-Pin_1): J3.1 (Pin_1), R3.2
Other:
- moved on the sheet: J1, J2, J3, J4, J5, R1, R3, TP7

Commit message: Updated board version to v1.1.1
Increased hole size from M2 to M3
Parts:
- H1, H2, H3, H4: footprint MountingHole:MountingHole_2.2mm_M2_Pad_Via -> MountingHole:MountingHole_3.2mm_M3_Pad_Via
Changed lines of the file:
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@@
 			)
 		)
-		(property "Footprint" "MountingHole:MountingHole_2.2mm_M2_Pad_Via"
+		(property "Footprint" "MountingHole:MountingHole_3.2mm_M3_Pad_Via"
 			(at 139.7 31.75 0)
 			(hide yes)
@@
 			)
 		)
-		(property "Footprint" "MountingHole:MountingHole_2.2mm_M2_Pad_Via"
+		(property "Footprint" "MountingHole:MountingHole_3.2mm_M3_Pad_Via"
 			(at 139.7 45.72 0)
 			(hide yes)
@@
 			)
 		)
-		(property "Footprint" "MountingHole:MountingHole_2.2mm_M2_Pad_Via"
+		(property "Footprint" "MountingHole:MountingHole_3.2mm_M3_Pad_Via"
 			(at 166.37 31.75 0)
 			(hide yes)
@@
 			)
 		)
-		(property "Footprint" "MountingHole:MountingHole_2.2mm_M2_Pad_Via"
+		(property "Footprint" "MountingHole:MountingHole_3.2mm_M3_Pad_Via"
 			(at 166.37 45.72 0)
 			(hide yes)
